File: pcb_ejemplo/pcb_ejemplo.kicad_sch (KiCad schematic)
At the start: 5 parts, among them J1 UPDI, U1 Microcontroller_ATtiny412_SSFR

Commit message: update PCB
Parts:
- R1: value 1 k -> 499 Ohm
Connections:
- net PWR_5V: now also J1.3 (Pin_3); no longer J1.1 (Pin_1)
- net UPDI: now also J1.1 (Pin_1); no longer J1.3 (Pin_3)
Changed lines of the file:
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@@
 (kicad_sch (version 20211123) (generator eeschema)
   (paper "A4")
+  (junction (at 153.416 90.678) (diameter 0) (color 0 0 0 0)
+  )
+  (junction (at 153.416 53.34) (diameter 0) (color 0 0 0 0)
+  )
   (no_connect (at 168.656 79.248))
   (no_connect (at 168.656 76.708))
   (no_connect (at 168.656 71.628))
   (no_connect (at 168.656 66.548))
-  (wire (pts (xy 153.416 89.408) (xy 153.416 91.694))
-    (stroke (width 0) (type default) (color 0 0 0 0))
-  )
-  (wire (pts (xy 153.416 52.324) (xy 153.416 53.848))
+  (wire (pts (xy 153.416 89.408) (xy 153.416 90.678))
+    (stroke (width 0) (type default) (color 0 0 0 0))
+  )
+  (wire (pts (xy 153.416 52.324) (xy 153.416 53.34))
+    (stroke (width 0) (type default) (color 0 0 0 0))
+  )
+  (wire (pts (xy 153.416 90.678) (xy 153.416 91.694))
     (stroke (width 0) (type default) (color 0 0 0 0))
   )
@@
   )
   (wire (pts (xy 191.516 35.052) (xy 198.374 35.052))
+    (stroke (width 0) (type default) (color 0 0 0 0))
+  )
+  (wire (pts (xy 153.416 53.34) (xy 153.416 53.848))
     (stroke (width 0) (type default) (color 0 0 0 0))
   )
@@
     )
   )
-  (global_label "UPDI" (shape input) (at 203.2 65.786 180) (fields_autoplaced)
+  (global_label "UPDI" (shape input) (at 201.93 70.866 180) (fields_autoplaced)
     (effects (font (size 1.27 1.27)) (justify right))
-    (property "Referencias entre hojas" "${INTERSHEET_REFS}" (id 0) (at 196.3117 65.7066 0)
+    (property "Referencias entre hojas" "${INTERSHEET_REFS}" (id 0) (at 195.0417 70.7866 0)
       (effects (font (size 1.27 1.27)) (justify right) hide)
     )
@@
     (pin "1")
   )
-  (symbol (lib_id "fab:PWR_5V") (at 201.93 70.866 90) (unit 1)
-    (in_bom yes) (on_board yes) (fields_autoplaced)
-    (property "Reference" "#PWR0106" (id 0) (at 205.74 70.866 0)
-      (effects (font (size 1.27 1.27)) hide)
-    )
-    (property "Value" "PWR_5V" (id 1) (at 198.12 70.8659 90)
+  (symbol (lib_id "fab:PWR_5V") (at 203.2 65.786 90) (unit 1)
+    (in_bom yes) (on_board yes) (fields_autoplaced)
+    (property "Reference" "#PWR0106" (id 0) (at 207.01 65.786 0)
+      (effects (font (size 1.27 1.27)) hide)
+    )
+    (property "Value" "PWR_5V" (id 1) (at 199.39 65.7859 90)
       (effects (font (size 1.27 1.27)) (justify left))
     )
-    (property "Footprint" "" (id 2) (at 201.93 70.866 0)
-      (effects (font (size 1.27 1.27)) hide)
-    )
-    (property "Datasheet" "" (id 3) (at 201.93 70.866 0)
+    (property "Footprint" "" (id 2) (at 203.2 65.786 0)
+      (effects (font (size 1.27 1.27)) hide)
+    )
+    (property "Datasheet" "" (id 3) (at 203.2 65.786 0)
       (effects (font (size 1.27 1.27)) hide)
     )
@@
     (in_bom yes) (on_board yes) (fields_autoplaced)
     (property "Reference" "R1" (id 0) (at 203.454 29.21 90))
-    (property "Value" "1 k" (id 1) (at 203.454 31.75 90))
+    (property "Value" "499 Ohm" (id 1) (at 203.454 31.75 90))
     (property "Footprint" "fab:R_1206" (id 2) (at 203.454 35.052 90)
       (effects (font (size 1.27 1.27)) hide)
@@
     (pin "2")
   )
+  (symbol (lib_id "power:PWR_FLAG") (at 153.416 53.34 90) (unit 1)
+    (in_bom yes) (on_board yes) (fields_autoplaced)
+    (property "Reference" "#FLG0102" (id 0) (at 151.511 53.34 0)
+      (effects (font (size 1.27 1.27)) hide)
+    )
+    (property "Value" "PWR_FLAG" (id 1) (at 150.114 53.3399 90)
+      (effects (font (size 1.27 1.27)) (justify left))
+    )
+    (property "Footprint" "" (id 2) (at 153.416 53.34 0)
+      (effects (font (size 1.27 1.27)) hide)
+    )
+    (property "Datasheet" "~" (id 3) (at 153.416 53.34 0)
+      (effects (font (size 1.27 1.27)) hide)
+    )
+    (pin "1")
+  )
   (symbol (lib_id "fab:PWR_GND") (at 153.416 91.694 0) (unit 1)
     (in_bom yes) (on_board yes) (fields_autoplaced)
@@
     (pin "2")
   )
+  (symbol (lib_id "power:PWR_FLAG") (at 153.416 90.678 90) (unit 1)
+    (in_bom yes) (on_board yes) (fields_autoplaced)
+    (property "Reference" "#FLG0101" (id 0) (at 151.511 90.678 0)
+      (effects (font (size 1.27 1.27)) hide)
+    )
+    (property "Value" "PWR_FLAG" (id 1) (at 149.86 90.6779 90)
+      (effects (font (size 1.27 1.27)) (justify left))
+    )
+    (property "Footprint" "" (id 2) (at 153.416 90.678 0)
+      (effects (font (size 1.27 1.27)) hide)
+    )
+    (property "Datasheet" "~" (id 3) (at 153.416 90.678 0)
+      (effects (font (size 1.27 1.27)) hide)
+    )
+    (pin "1")
+  )
   (sheet_instances
     (path "/" (page "1"))
   )
   (symbol_instances
+    (path "/fcb1d7e9-c34d-466a-82db-67752e576e95"
+      (reference "#FLG0101") (unit 1) (value "PWR_FLAG") (footprint "")
+    )
+    (path "/7a14b682-2294-4a3d-a35f-fc417ebba5b4"
+      (reference "#FLG0102") (unit 1) (value "PWR_FLAG") (footprint "")
+    )
     (path "/7e9e73f3-5b5f-4b51-a9f3-0d51c6a3a7e7"
       (reference "#PWR0101") (unit 1) (value "PWR_GND") (footprint "")
@@
     )
     (path "/5d6f4bcc-45fc-442f-8fab-4facdefbec3c"
-      (reference "R1") (unit 1) (value "1 k") (footprint "fab:R_1206")
+      (reference "R1") (unit 1) (value "499 Ohm") (footprint "fab:R_1206")
     )
     (path "/71de2cc1-3e10-4375-a452-3f562b56a7ab"
